Commit message: Created xacro files for the urdf model. Add .gitignore to skip VS Code and build files

File: src/my_robot_description/urdf/arm.xacro (robot description, xacro)
@@ -1,10 +1,4 @@
 <?xml version="1.0"?>
-<robot name="my_robot">
-    <material name="grey">
-        <color rgba="0.5 0.5 0.5 1" />
-    </material>
-    <material name="blue">
-        <color rgba="0 0 0.5 1" />
-    </material>
+<robot xmlns:xacro="http://wwww.ros.org/wiki/xacro">
     <link name="base_link">
         <visual>
